File: ELRS_Rx_4PWM_ESC_1S.kicad_pcb (KiCad board)
At the start: 4 copper layers, 20 x 20 mm, 83 parts, among them J1 Conn_Coaxial, J2 Conn_02x06_Counter_Clockwise, J5 Conn_Coaxial, Q1 UT6MA3, Q2 UT6MA3, Q3 UT6MA3, U1 SPX3819M5-L-3-3, U2 ESP8285, U3 NC7NZ14L8X, U4 EFM8BB21F16G-QFN20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

Commit message: V1.1 adjust pull-up resistors and layout
Parts:
- added R29: 10k, Resistor_SMD:R_0402_1005Metric, F.Cu at (169.6, 57.7)
- R13: value 10k -> 4k7
- moved R6 0.45 mm to (169.1, 56.2)
- moved R8 0.40 mm to (170.0, 56.2)
Connections:
- J5 pad 2: Net-(J5-Pad2) -> unconnected-(J5-Pad2)
- U2 pad 20: Net-(U2-Pad20) -> unconnected-(U2-Pad20)
- U2 pad 21: Net-(U2-Pad21) -> unconnected-(U2-Pad21)
- U2 pad 22: Net-(U2-Pad22) -> unconnected-(U2-Pad22)
- U2 pad 23: Net-(U2-Pad23) -> unconnected-(U2-Pad23)
- U2 pad 5: Net-(U2-Pad5) -> unconnected-(U2-Pad5)
- U4 pad 15: Net-(U4-Pad15) -> unconnected-(U4-Pad15)
- U4 pad 16: Net-(U4-Pad16) -> unconnected-(U4-Pad16)
- U4 pad 7: Net-(U4-Pad7) -> unconnected-(U4-Pad7)
- U6 pad 10: Net-(U6-Pad10) -> unconnected-(U6-Pad10)
- U6 pad 14: Net-(U6-Pad14) -> unconnected-(U6-Pad14)
- U6 pad 9: Net-(U6-Pad9) -> unconnected-(U6-Pad9)
Routing:
- net PWM2: track 5.24 -> 6.65 mm
- net +3V3: track 24.4 -> 25.3 mm
- net PWM4: track 6.31 -> 6.89 mm
- added copper zone on In1.Cu, net +3V3
- added copper zone on In1.Cu, net +BATT
- added copper zone on In2.Cu, net GND
- removed copper zone on In1.Cu_3V3, net +3V3
- removed copper zone on In1.Cu_3V3, net +BATT
- removed copper zone on In2.Cu_Gnd, net GND
Other:
- net class Default removed
- board text added: "rev 1.1"
- board text removed: "rev 1.0"
